Commit message: Controller input function, main logic in main.py

File: main.urdf (robot description, URDF)
Before this commit: robot simple_arm, 3 links, 2 joints
Links:
- link link1: geometry visual cylinder length=0.1403 radius=0.01
- link link2: geometry visual cylinder length=0.25 radius=0.01
Joints:
- joint joint2: origin xyz=0 0 0.3 rpy=0 0 0 -> xyz=0 0.04 0.05 rpy=0 0 0

Commit message: Changed the URDF, the arm has complicated geometry

File: main.urdf (robot description, URDF)
Before this commit: robot simple_arm, 3 links, 2 joints
Links:
- link link2: geometry visual cylinder length=0.16 radius=0.01
Joints:
- joint joint2: origin xyz=0 0.04 0.05 rpy=0 0 0 -> xyz=0.038 -0.045 0.1353 rpy=0 0 0
